Commit message: added robot launch script

File: turtlebot_description/urdf/sensors/hokuyo_laser.urdf.xacro (robot description, xacro)
@@ -12,6 +12,6 @@
       <origin xyz="0 0 0" rpy="0 0 0"/>
       <geometry>
-        <!--<box size="0.058 0.058 0.087"/>-->
-        <mesh filename="$(find turtlebot_description)/meshes/sensors/hokuyo_utm_30lx.dae"/>
+        <box size="0.058 0.058 0.087"/>
+        <!--<mesh filename="$(find turtlebot_description)/meshes/sensors/hokuyo_utm_30lx.dae"/>-->
       </geometry>
     </visual>
