Commit message: - clean up sensor

File: turtlebot_description/urdf/sensors/turtlebot_logical_dist.urdf.xacro (robot description, xacro)
@@ -4,5 +4,5 @@
   <xacro:macro name="turtlebot_logical_dist" params="parent orientation_z name">
   <joint name="${name}" type="fixed">
-    <origin xyz="0.00 0.00 0.4535" rpy="0 0 ${orientation_z}"/>
+    <origin xyz="0.00 0.00 0.4" rpy="0 0 ${orientation_z}"/>
     <parent link="${parent}" />
     <child link="${name}_link" />
@@ -12,5 +12,5 @@
       <origin xyz="0 0 0" rpy="0 0 0"/>
       <geometry>
-        <box size="0.058 0.058 0.087"/>
+        <box size="0.058 0.058 0.0001"/>
       </geometry>
     </visual>
@@ -20,10 +20,4 @@
       <inertia ixx="2.632e-4" ixy="0" ixz="0" iyy="2.632e-4" iyz="0" izz="1.62e-4"/>
     </inertial>
-    <collision>
-      <origin xyz="0 0 -0.0115" rpy="0 0 0"/>
-      <geometry>
-        <box size="0.058 0.058 0.087"/>
-      </geometry>
-    </collision>
   </link>
   <turtlebot_logical name="${name}"/>
