Commit message: - fixed msg package in doorcmd.sh => DoorCmd.msg moved from hinged_door_controller to ttb_msgs - lifted logical camera - fixed logical camera plugin

File: turtlebot_description/urdf/sensors/turtlebot_logical_camera_plugin.urdf.xacro (robot description, xacro)
@@ -4,5 +4,5 @@
   <xacro:macro name="turtlebot_logical_camera_plugin" params="parent orientation_z name">
   <joint name="${name}" type="fixed">
-    <origin xyz="0.00 0.00 0.4" rpy="0 0 ${orientation_z}"/>
+    <origin xyz="0.00 0.00 0.55" rpy="0 0 ${orientation_z}"/>
     <parent link="${parent}" />
     <child link="${name}_link" />

Commit message: working on logical camera

File: turtlebot_description/urdf/sensors/turtlebot_logical_camera_plugin.urdf.xacro (robot description, xacro)
@@ -4,15 +4,15 @@
   <xacro:macro name="turtlebot_logical_camera_plugin" params="parent orientation_z name">
   <joint name="${name}" type="fixed">
-    <origin xyz="0.00 0.00 0.55" rpy="0 0 ${orientation_z}"/>
+    <origin xyz="0.00 0.00 1.25" rpy="0 0 ${orientation_z}"/>
     <parent link="${parent}" />
     <child link="${name}_link" />
   </joint>
   <link name="${name}_link">
-    <visual>
+    <!--<visual>
       <origin xyz="0 0 0" rpy="0 0 0"/>
       <geometry>
         <box size="0.058 0.058 0.0001"/>
       </geometry>
-    </visual>
+    </visual>-->
   </link>
   <turtlebot_logical_camera name="${name}"/>
