Commit message: added logical camero to turtlebot

File: turtlebot_description/robots/kobuki_ninja-hexagons_ninja-kinect.urdf.xacro (robot description, xacro)
@@ -7,7 +7,9 @@
 <robot name="turtlebot" xmlns:xacro="http://ros.org/wiki/xacro">
   <xacro:include filename="$(find turtlebot_description)/urdf/turtlebot_library.urdf.xacro" />
+  <xacro:include filename="$(find turtlebot_description)/urdf/sensors/turtlebot_logical_dist.urdf.xacro"/>
   <kobuki/>
   <stack_ninja-hexagons parent="base_link"/>
   <sensor_ninja-kinect  parent="base_link"/>
   <sensor_hokuyo parent="base_link"/>
+  <turtlebot_logical_dist parent="base_link"/>
 </robot>

File: turtlebot_description/urdf/turtlebot_gazebo.urdf.xacro (robot description, xacro)
@@ -74,3 +74,24 @@
     </gazebo>
   </xacro:macro>
+  <!-- Logical Distance Sensor -->
+  <xacro:macro name="turtlebot_logical">
+    <gazebo reference="distance_link">
+      <sensor type="logical_camera" name="distance_sensor">
+        <always_on>true</always_on>
+        <update_rate>20.0</update_rate>
+        <camera>
+          <horizontal_fov>${2*M_PI}</horizontal_fov>
+          <clip>
+            <near>0.05</near>
+            <far>8.0</far>
+          </clip>
+        </camera>
+        <plugin name="turtlebot_gazebo_distance_sensor" filename="libturtlebot_gazebo_distance_sensor.so">
+          <cameraName>camera</cameraName>
+          <alwaysOn>true</alwaysOn>
+          <updateRate>10</updateRate>
+        </plugin>
+      </sensor>
+    </gazebo>
+  </xacro:macro>
 </robot>

Commit message: added second logical camera and rotated it backwards

File: turtlebot_description/robots/kobuki_ninja-hexagons_ninja-kinect.urdf.xacro (robot description, xacro)
@@ -13,3 +13,4 @@
   <sensor_hokuyo parent="base_link"/>
   <turtlebot_logical_dist parent="base_link"/>
+  <turtlebot_logical_dist2 parent="base_link"/>
 </robot>

File: turtlebot_description/urdf/sensors/turtlebot_logical_dist.urdf.xacro (robot description, xacro)
@@ -29,3 +29,30 @@
   <turtlebot_logical />
   </xacro:macro>
+  <xacro:macro name="turtlebot_logical_dist2" params="parent">
+  <joint name="logical_camera2" type="fixed">
+    <origin xyz="0.00 0.00 0.4535" rpy="0 0 ${M_PI}"/>
+    <parent link="${parent}" />
+    <child link="distance_link2" />
+  </joint>
+  <link name="distance_link2">
+    <visual>
+      <origin xyz="0 0 0" rpy="0 0 0"/>
+      <geometry>
+        <box size="0.058 0.058 0.087"/>
+      </geometry>
+    </visual>
+    <inertial>
+      <mass value="0.270"/>
+      <origin xyz="0 0 0" rpy="0 0 0"/>
+      <inertia ixx="2.632e-4" ixy="0" ixz="0" iyy="2.632e-4" iyz="0" izz="1.62e-4"/>
+    </inertial>
+    <collision>
+      <origin xyz="0 0 -0.0115" rpy="0 0 0"/>
+      <geometry>
+        <box size="0.058 0.058 0.087"/>
+      </geometry>
+    </collision>
+  </link>
+  <turtlebot_logical2 />
+  </xacro:macro>
 </robot>

File: turtlebot_description/urdf/turtlebot_gazebo.urdf.xacro (robot description, xacro)
@@ -81,5 +81,5 @@
         <update_rate>20.0</update_rate>
         <logical_camera>
-          <horizontal_fov>${2*M_PI}</horizontal_fov>
+          <horizontal_fov>${M_PI}</horizontal_fov>
           <near>0.05</near>
           <far>8.0</far>
@@ -90,5 +90,29 @@
           <updateRate>20</updateRate>
           <logical_camera>
-            <horizontal_fov>${2*M_PI}</horizontal_fov>
+            <horizontal_fov>${M_PI}</horizontal_fov>
+            <near>0.05</near>
+            <far>8.0</far>
+          </logical_camera>
+        </plugin>
+      </sensor>
+    </gazebo>
+  </xacro:macro>
+  <!-- Logical Distance Sensor2 -->
+  <xacro:macro name="turtlebot_logical2">
+    <gazebo reference="distance_link2">
+      <sensor type="logical_camera" name="distance_sensor">
+        <always_on>true</always_on>
+        <update_rate>20.0</update_rate>
+        <logical_camera>
+          <horizontal_fov>${M_PI}</horizontal_fov>
+          <near>0.05</near>
+          <far>8.0</far>
+          </logical_camera>
+        <plugin name="turtlebot_gazebo_distance_sensor" filename="libturtlebot_gazebo_distance_sensor.so">
+          <cameraName>camera</cameraName>
+          <alwaysOn>true</alwaysOn>
+          <updateRate>20</updateRate>
+          <logical_camera>
+            <horizontal_fov>${M_PI}</horizontal_fov>
             <near>0.05</near>
             <far>8.0</far>

Commit message: - created box for collecting boxes - cleanup logical camera xacros (introduced params)

File: turtlebot_description/robots/kobuki_ninja-hexagons_ninja-kinect.urdf.xacro (robot description, xacro)
@@ -7,10 +7,7 @@
 <robot name="turtlebot" xmlns:xacro="http://ros.org/wiki/xacro">
   <xacro:include filename="$(find turtlebot_description)/urdf/turtlebot_library.urdf.xacro" />
-  <!--<xacro:include filename="$(find turtlebot_description)/urdf/sensors/turtlebot_logical_dist.urdf.xacro"/> -->
   <kobuki/>
   <stack_ninja-hexagons parent="base_link"/>
   <sensor_ninja-kinect  parent="base_link"/>
   <sensor_hokuyo parent="base_link"/>
-  <!--<turtlebot_logical_dist parent="base_link"/>
-  <turtlebot_logical_dist2 parent="base_link"/>-->
 </robot>

File: turtlebot_description/robots/kobuki_ninja-hexagons_ninja-kinect_sim.urdf.xacro (robot description, xacro)
@@ -12,5 +12,5 @@
   <sensor_ninja-kinect  parent="base_link"/>
   <sensor_hokuyo parent="base_link"/>
-  <turtlebot_logical_dist parent="base_link"/>
-  <turtlebot_logical_dist2 parent="base_link"/>
+  <turtlebot_logical_dist name="sensor1" parent="base_link" orientation_z="0.0"/>
+  <turtlebot_logical_dist name="sensor2" parent="base_link" orientation_z="3.141"/>
 </robot>

File: turtlebot_description/urdf/sensors/hokuyo_laser.urdf.xacro (robot description, xacro)
@@ -12,6 +12,6 @@
       <origin xyz="0 0 0" rpy="0 0 0"/>
       <geometry>
-        <box size="0.058 0.058 0.087"/>
-        <!--<mesh filename="$(find turtlebot_description)/meshes/sensors/hokuyo_utm_30lx.dae"/>-->
+        <!--<box size="0.058 0.058 0.087"/> -->
+        <mesh filename="package://turtlebot_description/meshes/sensors/hokuyo_utm_30lx.dae"/>
       </geometry>
     </visual>

File: turtlebot_description/urdf/sensors/turtlebot_logical_dist.urdf.xacro (robot description, xacro)
@@ -2,11 +2,11 @@
 <robot name="turtlebot_logical_dist" xmlns:xacro="http://ros.org/wiki/xacro">
   <xacro:include filename="$(find turtlebot_description)/urdf/turtlebot_gazebo.urdf.xacro"/>
-  <xacro:macro name="turtlebot_logical_dist" params="parent">
-  <joint name="logical_camera" type="fixed">
-    <origin xyz="0.00 0.00 0.4535" rpy="0 0 0"/>
+  <xacro:macro name="turtlebot_logical_dist" params="parent orientation_z name">
+  <joint name="${name}" type="fixed">
+    <origin xyz="0.00 0.00 0.4535" rpy="0 0 ${orientation_z}"/>
     <parent link="${parent}" />
-    <child link="distance_link" />
+    <child link="${name}_link" />
   </joint>
-  <link name="distance_link">
+  <link name="${name}_link">
     <visual>
       <origin xyz="0 0 0" rpy="0 0 0"/>
@@ -27,32 +27,5 @@
     </collision>
   </link>
-  <turtlebot_logical />
-  </xacro:macro>
-  <xacro:macro name="turtlebot_logical_dist2" params="parent">
-  <joint name="logical_camera2" type="fixed">
-    <origin xyz="0.00 0.00 0.4535" rpy="0 0 ${M_PI}"/>
-    <parent link="${parent}" />
-    <child link="distance_link2" />
-  </joint>
-  <link name="distance_link2">
-    <visual>
-      <origin xyz="0 0 0" rpy="0 0 0"/>
-      <geometry>
-        <box size="0.058 0.058 0.087"/>
-      </geometry>
-    </visual>
-    <inertial>
-      <mass value="0.270"/>
-      <origin xyz="0 0 0" rpy="0 0 0"/>
-      <inertia ixx="2.632e-4" ixy="0" ixz="0" iyy="2.632e-4" iyz="0" izz="1.62e-4"/>
-    </inertial>
-    <collision>
-      <origin xyz="0 0 -0.0115" rpy="0 0 0"/>
-      <geometry>
-        <box size="0.058 0.058 0.087"/>
-      </geometry>
-    </collision>
-  </link>
-  <turtlebot_logical2 />
+  <turtlebot_logical name="${name}"/>
   </xacro:macro>
 </robot>

File: turtlebot_description/urdf/turtlebot_gazebo.urdf.xacro (robot description, xacro)
@@ -75,31 +75,7 @@
   </xacro:macro>
   <!-- Logical Distance Sensor -->
-  <xacro:macro name="turtlebot_logical">
-    <gazebo reference="distance_link">
-      <sensor type="logical_camera" name="distance_sensor">
-        <always_on>true</always_on>
-        <update_rate>20.0</update_rate>
-        <logical_camera>
-          <horizontal_fov>${M_PI}</horizontal_fov>
-          <near>0.05</near>
-          <far>8.0</far>
-          </logical_camera>
-        <plugin name="turtlebot_gazebo_distance_sensor" filename="libturtlebot_gazebo_distance_sensor.so">
-          <cameraName>camera</cameraName>
-          <alwaysOn>true</alwaysOn>
-          <updateRate>20</updateRate>
-          <logical_camera>
-            <horizontal_fov>${M_PI}</horizontal_fov>
-            <near>0.05</near>
-            <far>8.0</far>
-          </logical_camera>
-        </plugin>
-      </sensor>
-    </gazebo>
-  </xacro:macro>
-  <!-- Logical Distance Sensor2 -->
-  <xacro:macro name="turtlebot_logical2">
-    <gazebo reference="distance_link2">
-      <sensor type="logical_camera" name="distance_sensor">
+  <xacro:macro name="turtlebot_logical" params="name">
+    <gazebo reference="${name}_link">
+      <sensor type="logical_camera" name="distance_${name}">
         <always_on>true</always_on>
         <update_rate>20.0</update_rate>
