Commit message: -added arm link to turtlebot -added model plugin for arm -added two coke can to the world

File: turtlebot_description/robots/kobuki_ninja-hexagons_ninja-kinect_sim.urdf.xacro (robot description, xacro)
@@ -8,4 +8,5 @@
   <xacro:include filename="$(find turtlebot_description)/urdf/turtlebot_library.urdf.xacro" />
   <xacro:include filename="$(find turtlebot_description)/urdf/sensors/turtlebot_logical_dist.urdf.xacro"/>
+  <xacro:include filename="$(find turtlebot_description)/urdf/actuators/turtlebot_sim_arm.urdf.xacro"/>
   <kobuki/>
   <stack_ninja-hexagons parent="base_link"/>
@@ -14,3 +15,4 @@
   <turtlebot_logical_dist name="sensor1" parent="base_link" orientation_z="0.0"/>
   <turtlebot_logical_dist name="sensor2" parent="base_link" orientation_z="3.141"/>
+  <turtlebot_sim_arm name="arm" parent="base_link"/>
 </robot>

File: turtlebot_description/urdf/turtlebot_gazebo.urdf.xacro (robot description, xacro)
@@ -98,3 +98,10 @@
     </gazebo>
   </xacro:macro>
+  <!-- Turtlebot Arm -->
+  <xacro:macro name="turtlebot_arm" params="name">
+    <gazebo>
+            <plugin name="turtlebot_gazebo_arm" filename="libturtlebot_gazebo_arm.so">
+ 	    </plugin>
+    </gazebo>
+  </xacro:macro>
 </robot>

Commit message: - arm first working verison (horrible)

File: turtlebot_description/robots/kobuki_ninja-hexagons_ninja-kinect_sim.urdf.xacro (robot description, xacro)
@@ -15,4 +15,4 @@
   <turtlebot_logical_dist name="sensor1" parent="base_link" orientation_z="0.0"/>
   <turtlebot_logical_dist name="sensor2" parent="base_link" orientation_z="3.141"/>
-  <turtlebot_sim_arm name="arm" parent="base_link"/>
+  <turtlebot_sim_arm name="arm" parent="base_footprint"/>
 </robot>

File: turtlebot_description/urdf/actuators/turtlebot_sim_arm.urdf.xacro (robot description, xacro)
@@ -2,13 +2,13 @@
 <robot name="turtlebot_sim_arm" xmlns:xacro="http://ros.org/wiki/xacro">
   <xacro:include filename="$(find turtlebot_description)/urdf/turtlebot_gazebo.urdf.xacro"/>
-  <xacro:macro name="turtlebot_sim_arm" params="parent name">
-  <joint name="${name}" type="fixed">
+  <xacro:macro name="turtlebot_sim_arm" params="name parent">
+  <joint name="${name}" type="continuous">
     <origin xyz="0.00 0.00 0.5" rpy="0 0 0"/>
     <parent link="${parent}" />
     <child link="${name}_link" />
+    <axis xyz="0 0 1"/>
   </joint>
-  <link name="${name}_link">
-  </link>
-  <turtlebot_arm name="${name}"/>
+  <link name="${name}_link" />
+  <turtlebot_arm/>
   </xacro:macro>
 </robot>

File: turtlebot_description/urdf/turtlebot_gazebo.urdf.xacro (robot description, xacro)
@@ -99,8 +99,8 @@
   </xacro:macro>
   <!-- Turtlebot Arm -->
-  <xacro:macro name="turtlebot_arm" params="name">
+  <xacro:macro name="turtlebot_arm">
     <gazebo>
-            <plugin name="turtlebot_gazebo_arm" filename="libturtlebot_gazebo_arm.so">
- 	    </plugin>
+      <plugin name="turtlebot_gazebo_arm" filename="libturtlebot_gazebo_arm.so">
+      </plugin>
     </gazebo>
   </xacro:macro>

Commit message: - added logical occlusion camera - attached it to the ttb

File: turtlebot_description/robots/kobuki_ninja-hexagons_ninja-kinect_sim.urdf.xacro (robot description, xacro)
@@ -8,4 +8,5 @@
   <xacro:include filename="$(find turtlebot_description)/urdf/turtlebot_library.urdf.xacro" />
   <xacro:include filename="$(find turtlebot_description)/urdf/sensors/turtlebot_logical_dist.urdf.xacro"/>
+  <xacro:include filename="$(find turtlebot_description)/urdf/sensors/turtlebot_logical_occlusion_dist.urdf.xacro"/>
   <xacro:include filename="$(find turtlebot_description)/urdf/actuators/turtlebot_sim_arm.urdf.xacro"/>
   <kobuki/>
@@ -15,4 +16,5 @@
   <turtlebot_logical_dist name="sensor1" parent="base_link" orientation_z="0.0"/>
   <turtlebot_logical_dist name="sensor2" parent="base_link" orientation_z="3.141"/>
+  <turtlebot_logical_occlusion_dist name="sensor3" parent="base_link" orientation_z="0.0"/>
   <turtlebot_sim_arm name="arm" parent="base_footprint"/>
 </robot>

File: turtlebot_description/urdf/turtlebot_gazebo.urdf.xacro (robot description, xacro)
@@ -105,3 +105,22 @@
     </gazebo>
   </xacro:macro>
+ <!-- Logical occlusion Sensor -->
+  <xacro:macro name="turtlebot_logical_occlusion" params="name">
+    <gazebo reference="${name}_link">
+      <sensor type="logical_camera" name="logical_occlusion_camera_${name}">
+        <always_on>true</always_on>
+        <update_rate>20</update_rate>
+        <visualize>true</visualize>
+        <logical_camera>
+          <horizontal_fov>1.57</horizontal_fov>
+          <aspect_ratio>1</aspect_ratio>
+          <near>0.017</near>
+          <far>10</far>
+        </logical_camera>
+        <plugin name="logical_occlusion_plugin" filename="liblogical_occlusion_plugin.so">
+          <occluding_model>map_point</occluding_model>
+        </plugin>
+      </sensor>
+    </gazebo>
+  </xacro:macro>
 </robot>

Commit message: - some minor improvements for logical camera plugin - copied a lot of functionality from logical camera plugin to occlusion sensor

File: turtlebot_description/robots/kobuki_ninja-hexagons_ninja-kinect_sim.urdf.xacro (robot description, xacro)
@@ -17,4 +17,5 @@
   <turtlebot_logical_dist name="sensor2" parent="base_link" orientation_z="3.141"/>
   <turtlebot_logical_occlusion_dist name="sensor3" parent="base_link" orientation_z="0.0"/>
+  <turtlebot_logical_occlusion_dist name="sensor4" parent="base_link" orientation_z="3.141"/>
   <turtlebot_sim_arm name="arm" parent="base_footprint"/>
 </robot>

File: turtlebot_description/urdf/sensors/turtlebot_logical_occlusion_dist.urdf.xacro (robot description, xacro)
@@ -15,9 +15,4 @@
       </geometry>
     </visual>
-    <inertial>
-      <mass value="0.270"/>
-      <origin xyz="0 0 0" rpy="0 0 0"/>
-      <inertia ixx="2.632e-4" ixy="0" ixz="0" iyy="2.632e-4" iyz="0" izz="1.62e-4"/>
-    </inertial>
   </link>
   <turtlebot_logical_occlusion name="${name}"/>

File: turtlebot_description/urdf/turtlebot_gazebo.urdf.xacro (robot description, xacro)
@@ -84,5 +84,5 @@
           <near>0.05</near>
           <far>8.0</far>
-          </logical_camera>
+        </logical_camera>
         <plugin name="turtlebot_gazebo_distance_sensor" filename="libturtlebot_gazebo_distance_sensor.so">
           <cameraName>camera</cameraName>
@@ -111,14 +111,11 @@
         <always_on>true</always_on>
         <update_rate>20</update_rate>
-        <visualize>true</visualize>
         <logical_camera>
-          <horizontal_fov>1.57</horizontal_fov>
+          <horizontal_fov>${M_PI}</horizontal_fov>
           <aspect_ratio>1</aspect_ratio>
-          <near>0.017</near>
-          <far>10</far>
+          <near>0.15</near>
+          <far>8</far>
         </logical_camera>
-        <plugin name="logical_occlusion_plugin" filename="liblogical_occlusion_plugin.so">
-          <occluding_model>map_point</occluding_model>
-        </plugin>
+        <plugin name="logical_occlusion_plugin" filename="liblogical_occlusion_plugin.so"/>
       </sensor>
     </gazebo>

Commit message: renaming of logical occlusion camera bug fixes

File: turtlebot_description/robots/kobuki_ninja-hexagons_ninja-kinect_sim.urdf.xacro (robot description, xacro)
@@ -8,5 +8,5 @@
   <xacro:include filename="$(find turtlebot_description)/urdf/turtlebot_library.urdf.xacro" />
   <xacro:include filename="$(find turtlebot_description)/urdf/sensors/turtlebot_logical_dist.urdf.xacro"/>
-  <xacro:include filename="$(find turtlebot_description)/urdf/sensors/turtlebot_logical_occlusion_dist.urdf.xacro"/>
+  <xacro:include filename="$(find turtlebot_description)/urdf/sensors/turtlebot_logical_camera_plugin.urdf.xacro"/>
   <xacro:include filename="$(find turtlebot_description)/urdf/actuators/turtlebot_sim_arm.urdf.xacro"/>
   <kobuki/>
@@ -16,6 +16,6 @@
   <turtlebot_logical_dist name="sensor1" parent="base_link" orientation_z="0.0"/>
   <turtlebot_logical_dist name="sensor2" parent="base_link" orientation_z="3.141"/>
-  <turtlebot_logical_occlusion_dist name="sensor3" parent="base_link" orientation_z="0.0"/>
-  <turtlebot_logical_occlusion_dist name="sensor4" parent="base_link" orientation_z="3.141"/>
+  <turtlebot_logical_camera_plugin name="sensor3" parent="base_link" orientation_z="0.0"/>
+  <turtlebot_logical_camera_plugin name="sensor4" parent="base_link" orientation_z="3.141"/>
   <turtlebot_sim_arm name="arm" parent="base_footprint"/>
 </robot>

File: turtlebot_description/urdf/sensors/turtlebot_logical_camera_plugin.urdf.xacro (robot description, xacro)
@@ -2,5 +2,5 @@
 <robot name="turtlebot_logical_occlusion_dist" xmlns:xacro="http://ros.org/wiki/xacro">
   <xacro:include filename="$(find turtlebot_description)/urdf/turtlebot_gazebo.urdf.xacro"/>
-  <xacro:macro name="turtlebot_logical_occlusion_dist" params="parent orientation_z name">
+  <xacro:macro name="turtlebot_logical_camera_plugin" params="parent orientation_z name">
   <joint name="${name}" type="fixed">
     <origin xyz="0.00 0.00 0.4" rpy="0 0 ${orientation_z}"/>
@@ -16,5 +16,5 @@
     </visual>
   </link>
-  <turtlebot_logical_occlusion name="${name}"/>
+  <turtlebot_logical_camera name="${name}"/>
   </xacro:macro>
 </robot>

File: turtlebot_description/urdf/turtlebot_gazebo.urdf.xacro (robot description, xacro)
@@ -106,7 +106,7 @@
   </xacro:macro>
  <!-- Logical occlusion Sensor -->
-  <xacro:macro name="turtlebot_logical_occlusion" params="name">
+  <xacro:macro name="turtlebot_logical_camera" params="name">
     <gazebo reference="${name}_link">
-      <sensor type="logical_camera" name="logical_occlusion_camera_${name}">
+      <sensor type="logical_camera" name="logical_occlusion_camera_plugin_${name}">
         <always_on>true</always_on>
         <update_rate>20</update_rate>
@@ -114,8 +114,8 @@
           <horizontal_fov>${M_PI}</horizontal_fov>
           <aspect_ratio>1</aspect_ratio>
-          <near>0.15</near>
-          <far>8</far>
+          <near>0.20</near>
+          <far>8.0</far>
         </logical_camera>
-        <plugin name="logical_occlusion_plugin" filename="liblogical_occlusion_plugin.so"/>
+        <plugin name="turtlebot_gazebo_logical_camera" filename="libturtlebot_gazebo_logical_camera.so"/>
       </sensor>
     </gazebo>

Commit message: - removed muxer, safety-controller, smoother - fixed fake_localisation with extra plugin in gazebo

File: turtlebot_description/robots/kobuki_ninja-hexagons_ninja-kinect_sim.urdf.xacro (robot description, xacro)
@@ -19,3 +19,4 @@
   <turtlebot_logical_camera_plugin name="sensor2" parent="base_link" orientation_z="3.141"/>
   <turtlebot_sim_arm name="arm" parent="base_footprint"/>
+  <turtlebot_ground_truth_pose/>
 </robot>

File: turtlebot_description/urdf/turtlebot_gazebo.urdf.xacro (robot description, xacro)
@@ -121,3 +121,17 @@
     </gazebo>
   </xacro:macro>
+  <!-- Makes Gazebo publishing a ground truth position. -->
+  <xacro:macro name="turtlebot_ground_truth_pose">
+    <gazebo>
+      <plugin name="p3d_controller" filename="libgazebo_ros_p3d.so">
+       <alwaysOn>true</alwaysOn>
+       <updateRate>100.0</updateRate>
+       <bodyName>base_link</bodyName>
+       <topicName>ground_truth_pose</topicName>
+       <frameName>/map</frameName>
+       <xyzOffsets>1 1 0</xyzOffsets> <!-- option to initialize odometry for fake localization-->
+       <rpyOffsets>0 0 0</rpyOffsets>
+      </plugin>
+    </gazebo>
+  </xacro:macro>
 </robot>

Commit message: debug

File: turtlebot_description/robots/kobuki_ninja-hexagons_ninja-kinect_sim.urdf.xacro (robot description, xacro)
@@ -6,6 +6,5 @@
 -->
 <robot name="turtlebot" xmlns:xacro="http://ros.org/wiki/xacro">
-  <xacro:include filename="$(find turtlebot_description)/urdf/turtlebot_library.urdf.xacro" />
-  <!--<xacro:include filename="$(find turtlebot_description)/urdf/sensors/turtlebot_logical_dist.urdf.xacro"/>-->
+  <xacro:include filename="$(find turtlebot_description)/urdf/turtlebot_library.urdf.xacro"/>
   <xacro:include filename="$(find turtlebot_description)/urdf/sensors/turtlebot_logical_camera_plugin.urdf.xacro"/>
   <xacro:include filename="$(find turtlebot_description)/urdf/actuators/turtlebot_sim_arm.urdf.xacro"/>
@@ -14,6 +13,4 @@
   <sensor_ninja-kinect  parent="base_link"/>
   <sensor_hokuyo parent="base_link"/>
-  <!--<turtlebot_logical_dist name="sensor1" parent="base_link" orientation_z="0.0"/>
-  <turtlebot_logical_dist name="sensor2" parent="base_link" orientation_z="3.141"/> -->
   <turtlebot_logical_camera_plugin name="sensor1" parent="base_link" orientation_z="0.0"/>
   <turtlebot_logical_camera_plugin name="sensor2" parent="base_link" orientation_z="3.141"/>

File: turtlebot_description/urdf/turtlebot_gazebo.urdf.xacro (robot description, xacro)
@@ -74,28 +74,4 @@
     </gazebo>
   </xacro:macro>
-  <!-- Logical Distance Sensor -->
-  <xacro:macro name="turtlebot_logical" params="name">
-    <gazebo reference="${name}_link">
-      <sensor type="logical_camera" name="distance_${name}">
-        <always_on>true</always_on>
-        <update_rate>20.0</update_rate>
-        <logical_camera>
-          <horizontal_fov>${M_PI}</horizontal_fov>
-          <near>0.05</near>
-          <far>8.0</far>
-        </logical_camera>
-        <plugin name="turtlebot_gazebo_distance_sensor" filename="libturtlebot_gazebo_distance_sensor.so">
-          <cameraName>camera</cameraName>
-          <alwaysOn>true</alwaysOn>
-          <updateRate>20</updateRate>
-          <logical_camera>
-            <horizontal_fov>${M_PI}</horizontal_fov>
-            <near>0.05</near>
-            <far>8.0</far>
-          </logical_camera>
-        </plugin>
-      </sensor>
-    </gazebo>
-  </xacro:macro>
   <!-- Turtlebot Arm -->
   <xacro:macro name="turtlebot_arm">
@@ -105,5 +81,5 @@
     </gazebo>
   </xacro:macro>
- <!-- Logical occlusion Sensor -->
+ <!-- Logical Camera Sensor -->
   <xacro:macro name="turtlebot_logical_camera" params="name">
     <gazebo reference="${name}_link">

Commit message: - removed second logical camera sensor - changed plugin type sensor => model - refactoring

File: turtlebot_description/robots/kobuki_ninja-hexagons_ninja-kinect_sim.urdf.xacro (robot description, xacro)
@@ -14,5 +14,5 @@
   <sensor_hokuyo parent="base_link"/>
   <turtlebot_logical_camera_plugin name="sensor1" parent="base_link" orientation_z="0.0"/>
-  <turtlebot_logical_camera_plugin name="sensor2" parent="base_link" orientation_z="3.141"/>
+  <!--<turtlebot_logical_camera_plugin name="sensor2" parent="base_link" orientation_z="3.141"/>-->
   <turtlebot_sim_arm name="arm" parent="base_footprint"/>
   <turtlebot_ground_truth_pose/>

File: turtlebot_description/urdf/turtlebot_gazebo.urdf.xacro (robot description, xacro)
@@ -81,5 +81,5 @@
     </gazebo>
   </xacro:macro>
- <!-- Logical Camera Sensor -->
+ <!-- Logical Camera Sensor
   <xacro:macro name="turtlebot_logical_camera" params="name">
     <gazebo reference="${name}_link">
@@ -96,5 +96,10 @@
       </sensor>
     </gazebo>
-  </xacro:macro>
+  </xacro:macro> -->
+  <xacro:macro name="turtlebot_logical_camera" params="name">
+	<gazebo>
+      <plugin name="turtlebot_gazebo_logical_camera" filename="libturtlebot_gazebo_logical_camera.so"/>
+    </gazebo>
+  </xacro:macro> -->
   <!-- Makes Gazebo publishing a ground truth position. -->
   <xacro:macro name="turtlebot_ground_truth_pose">

Commit message: - adaptions

File: turtlebot_description/robots/kobuki_ninja-hexagons_ninja-kinect_sim.urdf.xacro (robot description, xacro)
@@ -6,4 +6,5 @@
 -->
 <robot name="turtlebot" xmlns:xacro="http://ros.org/wiki/xacro">
+  <xacro:arg name="robotNamespace" default="leonardo"/>
   <xacro:include filename="$(find turtlebot_description)/urdf/turtlebot_library.urdf.xacro"/>
   <xacro:include filename="$(find turtlebot_description)/urdf/sensors/turtlebot_logical_camera_plugin.urdf.xacro"/>
@@ -15,5 +16,5 @@
   <turtlebot_logical_camera_plugin name="logical_camera" parent="base_link" orientation_z="0.0"/>
   <turtlebot_sim_arm name="arm" parent="base_footprint"/>
-  <turtlebot_ground_truth_pose/>
+  <turtlebot_ground_truth_pose robotNamespace="$(arg robotNamespace)"/>
   <!--<gazebo>
  The plugin that determines the closest POI to a certain coordinate.

File: turtlebot_description/urdf/turtlebot_gazebo.urdf.xacro (robot description, xacro)
@@ -103,8 +103,9 @@
   </xacro:macro>
   <!-- Makes Gazebo publishing a ground truth position. -->
-  <xacro:macro name="turtlebot_ground_truth_pose">
+  <xacro:macro name="turtlebot_ground_truth_pose" params="robotNamespace">
     <gazebo>
       <plugin name="p3d_controller" filename="libgazebo_ros_p3d.so">
        <alwaysOn>true</alwaysOn>
+       <robotNamespace>${robotNamespace}</robotNamespace>
        <updateRate>100.0</updateRate>
        <bodyName>base_link</bodyName>

File: turtlebot_description/urdf/turtlebot_library.urdf.xacro (robot description, xacro)
@@ -8,5 +8,5 @@
   <xacro:include filename="$(find turtlebot_description)/urdf/turtlebot_properties.urdf.xacro"/><!-- Defines the position of the Kinect -->
   <!-- Bases -->
-  <xacro:include filename="$(find create_description)/urdf/create.urdf.xacro"/>
+  <!--<xacro:include filename="$(find create_description)/urdf/create.urdf.xacro"/>-->
   <xacro:include filename="$(find kobuki_description)/urdf/kobuki.urdf.xacro"/>
   <!-- Stacks -->
