Commit message: - fixed joint type

File: turtlebot_description/urdf/actuators/turtlebot_sim_arm.urdf.xacro (robot description, xacro)
@@ -3,5 +3,5 @@
   <xacro:include filename="$(find turtlebot_description)/urdf/turtlebot_gazebo.urdf.xacro"/>
   <xacro:macro name="turtlebot_sim_arm" params="name parent">
-  <joint name="${name}" type="continuous">
+  <joint name="${name}" type="fixed">
     <origin xyz="0.00 0.00 0.5" rpy="0 0 0"/>
     <parent link="${parent}" />
