Commit message: update

File: turtlebot_description/urdf/turtlebot_gazebo.urdf.xacro (robot description, xacro)
@@ -40,3 +40,37 @@
     </gazebo>
   </xacro:macro>
+  <!-- Hokuyo LIDAR for simulation -->
+  <xacro:macro name="hokuyo_laser">
+    <gazebo reference="base_laser_link">
+      <sensor type="ray" name="laser">
+        <pose>0 0 0 0 0 0</pose>
+        <visualize>false</visualize>
+        <update_rate>30</update_rate>
+        <ray>
+          <scan>
+            <horizontal>
+              <samples>1080</samples>
+              <resolution>1</resolution>
+              <min_angle>-2,3562</min_angle>
+              <max_angle>2,3562</max_angle>
+            </horizontal>
+          </scan>
+          <range>
+            <min>0.08</min>
+            <max>30.0</max>
+            <resolution>0.01</resolution>
+          </range>
+          <noise>
+            <type>gaussian</type>
+            <mean>0.0</mean>
+            <stddev>0.004</stddev>
+          </noise>
+        </ray>
+        <plugin name="hokuyo_node" filename="libgazebo_ros_laser.so">
+          <topicName>scan_hokuyo</topicName>
+          <frameName>base_laser_link</frameName>
+        </plugin>
+      </sensor>
+    </gazebo>
+  </xacro:macro>
 </robot>

File: turtlebot_description/urdf/turtlebot_library.urdf.xacro (robot description, xacro)
@@ -6,16 +6,20 @@
   <!-- General -->
   <xacro:include filename="$(find turtlebot_description)/urdf/common_properties.urdf.xacro"/>
-  <xacro:include filename="$(find turtlebot_description)/urdf/turtlebot_properties.urdf.xacro"/>
+  <xacro:include filename="$(find turtlebot_description)/urdf/turtlebot_properties.urdf.xacro"/><!-- Defines the position of the Kinect -->
   <!-- Bases -->
   <xacro:include filename="$(find create_description)/urdf/create.urdf.xacro"/>
-  <xacro:include filename="$(find kobuki_description)/urdf/kobuki.urdf.xacro" />
+  <xacro:include filename="$(find kobuki_description)/urdf/kobuki.urdf.xacro"/>
   <!-- Stacks -->
   <xacro:include filename="$(find turtlebot_description)/urdf/stacks/circles.urdf.xacro"/>
   <xacro:include filename="$(find turtlebot_description)/urdf/stacks/hexagons.urdf.xacro"/>
+  <xacro:include filename="$(find turtlebot_description)/urdf/stacks/ninja-hexagons.urdf.xacro"/>
   <!-- 3D Sensors -->
-  <xacro:include filename="$(find turtlebot_description)/urdf/sensors/kinect.urdf.xacro"/>
+  <!-- <xacro:include filename="$(find turtlebot_description)/urdf/sensors/kinect.urdf.xacro"/>-->
+  <xacro:include filename="$(find turtlebot_description)/urdf/sensors/ninja_kinect.urdf.xacro"/>
   <xacro:include filename="$(find turtlebot_description)/urdf/sensors/asus_xtion_pro.urdf.xacro"/>
   <xacro:include filename="$(find turtlebot_description)/urdf/sensors/asus_xtion_pro_offset.urdf.xacro"/>
   <xacro:include filename="$(find turtlebot_description)/urdf/sensors/astra.urdf.xacro"/>
   <xacro:include filename="$(find turtlebot_description)/urdf/sensors/r200.urdf.xacro"/>
+  <!-- 2D Sensors -->
+  <xacro:include filename="$(find turtlebot_description)/urdf/sensors/hokuyo_laser.urdf.xacro"/>
 </robot>

File: turtlebot_description/urdf/turtlebot_properties.urdf.xacro (robot description, xacro)
@@ -19,9 +19,15 @@
      (currently in development and awaiting feedback)
    -->
-	<xacro:property name="cam_px" value="-0.087" />
+<!--	<xacro:property name="cam_px" value="-0.087" /> -->
 <!--	<xacro:property name="cam_py" value="-0.0125" /> Y varies for different configurations. get sets in sensors_urdf -->
-	<xacro:property name="cam_pz" value="0.2870" />
-	<xacro:property name="cam_or" value="0" />
-	<xacro:property name="cam_op" value="0" />
-	<xacro:property name="cam_oy" value="0" />
+<!--	<xacro:property name="cam_pz" value="0.2870" /> -->
+<!--	<xacro:property name="cam_or" value="0" /> -->
+<!--	<xacro:property name="cam_op" value="0" /> -->
+<!--	<xacro:property name="cam_oy" value="0" /> -->
+  <xacro:property name="cam_px" value="0.08"/>
+  <!--<xacro:property name="cam_py" value="-0.0125" /> Y varies for different configurations. get sets in sensors_urdf -->
+  <xacro:property name="cam_pz" value="0.35"/>
+  <xacro:property name="cam_or" value="${M_PI}"/>
+  <xacro:property name="cam_op" value="${M_PI/8}"/>
+  <xacro:property name="cam_oy" value="0"/>
 </robot>

Commit message: - trying arround stuff

File: turtlebot_description/urdf/turtlebot_gazebo.urdf.xacro (robot description, xacro)
@@ -101,5 +101,5 @@
       <plugin name="turtlebot_gazebo_logical_camera" filename="libturtlebot_gazebo_logical_camera.so"/>
     </gazebo>
-  </xacro:macro> -->
+  </xacro:macro>
   <!-- Makes Gazebo publishing a ground truth position. -->
   <xacro:macro name="turtlebot_ground_truth_pose">
